File: Moisture-Sensor.sch (KiCad schematic (older format))
At the start: 3 parts, among them J4 INPUT

Commit message: fixed up some mistakes
Parts:
- C8: LCSC (none) -> C30926
- R10: LCSC (none) -> C25197
Changed lines of the file:
@@
 F 3 "~" H 5400 3550 50  0001 C CNN
 F 4 "C25197" H 5400 3550 50  0001 C CNN "LCSC PART #"
+F 5 "C25197" H 5400 3550 50  0001 C CNN "LCSC"
 	1    5400 3550
 	0    -1   1    0
@@
 F 3 "~" H 5750 3700 50  0001 C CNN
 F 4 "C30926" H 5750 3700 50  0001 C CNN "LCSC PART #"
+F 5 "C30926" H 5750 3700 50  0001 C CNN "LCSC"
 	1    5750 3700
 	-1   0    0    -1
