File: PMOS-Driver.sch (KiCad schematic (older format))
At the start: 4 parts, among them J3 Power, Q2 AO3401A

Commit message: fixed up some mistakes
Parts:
- D5: LCSC (none) -> C64982
- Q2: LCSC (none) -> C2997136
- R4: LCSC (none) -> C25197
Changed lines of the file:
@@
 F 3 "~" H 5350 3550 50  0001 C CNN
 F 4 "C25197" H 5350 3550 50  0001 C CNN "LCSC PART #"
+F 5 "C25197" H 5350 3550 50  0001 C CNN "LCSC"
 	1    5350 3550
 	0    1    1    0
@@
 F 3 "http://www.aosmd.com/pdfs/datasheet/AO3401A.pdf" H 5800 3550 50  0001 L CNN
 F 4 "C2997136" H 5800 3550 50  0001 C CNN "LCSC PART #"
+F 5 "C2997136" H 5800 3550 50  0001 C CNN "LCSC"
 	1    5800 3550
 	1    0    0    1
@@
 F 3 "~" V 5450 4000 50  0001 C CNN
 F 4 "C64982" H 5450 4000 50  0001 C CNN "LCSC PART #"
+F 5 "C64982" H 5450 4000 50  0001 C CNN "LCSC"
 	1    5450 4000
 	0    1    1    0
