File: power.sch (KiCad schematic (older format))
At the start: 12 parts

Commit message: added 3d model
Parts:
- removed D?: D_Zener, symbol Device:D_Zener
- removed F?: 3A, Fuse:Fuse_1206_3216Metric, symbol Device:Fuse
- removed Q?: AO3401A, Package_TO_SOT_SMD:SOT-23, symbol Transistor_FET:AO3401A
- removed R?: 10k, symbol Device:R_Small
- C3: renamed from C?; LCSC PART # (none) -> C96446
- C4: renamed from C?; LCSC PART # (none) -> C57112
- C6: renamed from C?; footprint Capacitor_SMD:C_0603_1608Metric -> Capacitor_Tantalum_SMD:CP_EIA-3528-21_Kemet-B; LCSC PART # (none) -> C16133
- D4: renamed from D?; footprint Diode_SMD:D_SMC -> Diode_SMD:D_SMA; LCSC PART # (none) -> C64982
- L1: renamed from L?; footprint (none) -> Inductor_SMD:L_0805_2012Metric; LCSC PART # (none) -> C32375
- R12: renamed from R?; footprint (none) -> Resistor_SMD:R_0603_1608Metric; LCSC PART # (none) -> C25197
- R13: renamed from R?; value 5.9k -> 5.6k; footprint (none) -> Resistor_SMD:R_0603_1608Metric; LCSC PART # (none) -> C23189
- U2: renamed from U?; LCSC PART # (none) -> C9864
Connections:
- net VIN: now also C3.1, U2.7 (VIN)
Changed lines of the file:
@@
 $Descr A4 11693 8268
 encoding utf-8
-Sheet 2 2
+Sheet 2 6
 Title ""
 Date ""
@@
 $EndDescr
 $Comp
-L Device:Fuse F?
-U 1 1 62DDDB40
-P 2750 2550
-F 0 "F?" V 2650 2550 50  0000 C CNN
-F 1 "3A" V 2850 2550 50  0000 C CNN
-F 2 "Fuse:Fuse_1206_3216Metric" V 2680 2550 50  0001 C CNN
-F 3 "~" H 2750 2550 50  0001 C CNN
-	1    2750 2550
-	0    1    1    0
-$EndComp
-$Comp
-L Regulator_Switching:TPS5430DDA U?
-U 1 1 62DE4279
-P 5850 2750
-F 0 "U?" H 5850 3217 50  0000 C CNN
-F 1 "TPS5430DDA" H 5850 3126 50  0000 C CNN
-F 2 "Package_SO:TI_SO-PowerPAD-8_ThermalVias" H 5900 2400 50  0001 L CIN
-F 3 "http://www.ti.com/lit/ds/symlink/tps5430.pdf" H 5850 2750 50  0001 C CNN
-	1    5850 2750
-	1    0    0    -1
-$EndComp
-$Comp
-L power:GND #PWR?
+L power:GND #PWR0133
 U 1 1 62DE4EA6
 P 5800 3200
-F 0 "#PWR?" H 5800 2950 50  0001 C CNN
+F 0 "#PWR0133" H 5800 2950 50  0001 C CNN
 F 1 "GND" H 5805 3027 50  0000 C CNN
 F 2 "" H 5800 3200 50  0001 C CNN
@@
 P 4850 2800
 AR Path="/62DE6325" Ref="C?"  Part="1"
-AR Path="/62D8A179/62DE6325" Ref="C?"  Part="1"
-F 0 "C?" H 4950 2850 50  0000 L CNN
+AR Path="/62D8A179/62DE6325" Ref="C3"  Part="1"
+F 0 "C3" H 4950 2850 50  0000 L CNN
 F 1 "10u" H 4950 2750 50  0000 L CNN
 F 2 "Capacitor_SMD:C_0603_1608Metric" H 4850 2800 50  0001 C CNN
 F 3 "~" H 4850 2800 50  0001 C CNN
+F 4 "C96446" H 4850 2800 50  0001 C CNN "LCSC PART #"
 	1    4850 2800
 	1    0    0    -1
 $EndComp
 $Comp
-L power:GND #PWR?
+L power:GND #PWR0134
 U 1 1 62DE6C42
 P 4850 3200
-F 0 "#PWR?" H 4850 2950 50  0001 C CNN
+F 0 "#PWR0134" H 4850 2950 50  0001 C CNN
 F 1 "GND" H 4855 3027 50  0000 C CNN
 F 2 "" H 4850 3200 50  0001 C CNN
@@
 P 6700 2550
 AR Path="/62DEB99C" Ref="C?"  Part="1"
-AR Path="/62D8A179/62DEB99C" Ref="C?"  Part="1"
-F 0 "C?" V 6550 2400 50  0000 L CNN
+AR Path="/62D8A179/62DEB99C" Ref="C4"  Part="1"
+F 0 "C4" V 6550 2400 50  0000 L CNN
 F 1 "10n" V 6550 2600 50  0000 L CNN
 F 2 "Capacitor_SMD:C_0603_1608Metric" H 6700 2550 50  0001 C CNN
 F 3 "~" H 6700 2550 50  0001 C CNN
+F 4 "C57112" H 6700 2550 50  0001 C CNN "LCSC PART #"
 	1    6700 2550
 	0    1    1    0
@@
 	6350 2750 7000 2750
 $Comp
-L Device:R_Small R?
+L Device:R_Small R12
 U 1 1 62DEF185
 P 8500 2950
-F 0 "R?" H 8559 2996 50  0000 L CNN
+F 0 "R12" H 8559 2996 50  0000 L CNN
 F 1 "10k" H 8559 2905 50  0000 L CNN
-F 2 "" H 8500 2950 50  0001 C CNN
+F 2 "Resistor_SMD:R_0603_1608Metric" H 8500 2950 50  0001 C CNN
 F 3 "~" H 8500 2950 50  0001 C CNN
+F 4 "C25197" H 8500 2950 50  0001 C CNN "LCSC PART #"
 	1    8500 2950
 	1    0    0    -1
 $EndComp
 $Comp
-L Device:R_Small R?
+L Device:R_Small R13
 U 1 1 62DF1415
 P 8500 3450
-F 0 "R?" H 8559 3496 50  0000 L CNN
-F 1 "5.9k" H 8559 3405 50  0000 L CNN
-F 2 "" H 8500 3450 50  0001 C CNN
+F 0 "R13" H 8559 3496 50  0000 L CNN
+F 1 "5.6k" H 8559 3405 50  0000 L CNN
+F 2 "Resistor_SMD:R_0603_1608Metric" H 8500 3450 50  0001 C CNN
 F 3 "~" H 8500 3450 50  0001 C CNN
+F 4 "C23189" H 8500 3450 50  0001 C CNN "LCSC PART #"
 	1    8500 3450
 	1    0    0    -1
 $EndComp
-Wire Wire Line
-	8500 3250 8500 3050
-Wire Wire Line
-	8500 3250 8500 3350
-Connection ~ 8500 3250
 $Comp
 L power:GND #PWR?
@@
 P 8500 3650
 AR Path="/62DF2783" Ref="#PWR?"  Part="1"
-AR Path="/62D8A179/62DF2783" Ref="#PWR?"  Part="1"
-F 0 "#PWR?" H 8500 3400 50  0001 C CNN
+AR Path="/62D8A179/62DF2783" Ref="#PWR0135"  Part="1"
+F 0 "#PWR0135" H 8500 3400 50  0001 C CNN
 F 1 "GND" H 8505 3477 50  0000 C CNN
 F 2 "" H 8500 3650 50  0001 C CNN
@@
 NoConn ~ 5350 2950
 $Comp
-L Diode:B340 D?
+L Diode:B340 D4
 U 1 1 62DFD261
 P 7350 2750
-F 0 "D?" V 7304 2829 50  0000 L CNN
+F 0 "D4" V 7304 2829 50  0000 L CNN
 F 1 "B340" V 7395 2829 50  0000 L CNN
-F 2 "Diode_SMD:D_SMC" H 7350 2575 50  0001 C CNN
+F 2 "Diode_SMD:D_SMA" H 7350 2575 50  0001 C CNN
 F 3 "http://www.jameco.com/Jameco/Products/ProdDS/1538777.pdf" H 7350 2750 50  0001 C CNN
+F 4 "C64982" H 7350 2750 50  0001 C CNN "LCSC PART #"
 	1    7350 2750
 	0    1    1    0
 $EndComp
-Wire Wire Line
-	6350 3250 6350 2950
-Wire Wire Line
-	6350 3250 8500 3250
 $Comp
 L power:GND #PWR?
@@
 P 7350 2950
 AR Path="/62E05321" Ref="#PWR?"  Part="1"
-AR Path="/62D8A179/62E05321" Ref="#PWR?"  Part="1"
-F 0 "#PWR?" H 7350 2700 50  0001 C CNN
+AR Path="/62D8A179/62E05321" Ref="#PWR0136"  Part="1"
+F 0 "#PWR0136" H 7350 2700 50  0001 C CNN
 F 1 "GND" H 7355 2777 50  0000 C CNN
 F 2 "" H 7350 2950 50  0001 C CNN
@@
 Connection ~ 7000 2550
 $Comp
-L Device:L_Small L?
+L Device:L_Small L1
 U 1 1 62E0858B
 P 7800 2550
-F 0 "L?" V 7985 2550 50  0000 C CNN
+F 0 "L1" V 7985 2550 50  0000 C CNN
 F 1 "L_Small" V 7894 2550 50  0000 C CNN
-F 2 "" H 7800 2550 50  0001 C CNN
+F 2 "Inductor_SMD:L_0805_2012Metric" H 7800 2550 50  0001 C CNN
 F 3 "~" H 7800 2550 50  0001 C CNN
+F 4 "C32375" H 7800 2550 50  0001 C CNN "LCSC PART #"
 	1    7800 2550
 	0    -1   -1   0
@@
 P 8100 2750
 AR Path="/62E08F95" Ref="C?"  Part="1"
-AR Path="/62D8A179/62E08F95" Ref="C?"  Part="1"
-F 0 "C?" H 8200 2800 50  0000 L CNN
+AR Path="/62D8A179/62E08F95" Ref="C6"  Part="1"
+F 0 "C6" H 8200 2800 50  0000 L CNN
 F 1 "100u" H 8200 2700 50  0000 L CNN
-F 2 "Capacitor_SMD:C_0603_1608Metric" H 8100 2750 50  0001 C CNN
+F 2 "Capacitor_Tantalum_SMD:CP_EIA-3528-21_Kemet-B" H 8100 2750 50  0001 C CNN
 F 3 "~" H 8100 2750 50  0001 C CNN
+F 4 "C16133" H 8100 2750 50  0001 C CNN "LCSC PART #"
 	1    8100 2750
 	1    0    0    -1
@@
 P 8100 2950
 AR Path="/62E0A027" Ref="#PWR?"  Part="1"
-AR Path="/62D8A179/62E0A027" Ref="#PWR?"  Part="1"
-F 0 "#PWR?" H 8100 2700 50  0001 C CNN
+AR Path="/62D8A179/62E0A027" Ref="#PWR0139"  Part="1"
+F 0 "#PWR0139" H 8100 2700 50  0001 C CNN
 F 1 "GND" H 8105 2777 50  0000 C CNN
 F 2 "" H 8100 2950 50  0001 C CNN
@@
 Wire Wire Line
 	8900 2550 8500 2550
-Text HLabel 2100 2550 0    50   Input ~ 0
+Text HLabel 4300 2550 0    50   Input ~ 0
 VIN
 Wire Wire Line
-	2100 2550 2600 2550
-$Comp
-L Transistor_FET:AO3401A Q?
-U 1 1 62E3CDA4
-P 3850 2650
-F 0 "Q?" V 4192 2650 50  0000 C CNN
-F 1 "AO3401A" V 4101 2650 50  0000 C CNN
-F 2 "Package_TO_SOT_SMD:SOT-23" H 4050 2575 50  0001 L CIN
-F 3 "http://www.aosmd.com/pdfs/datasheet/AO3401A.pdf" H 3850 2650 50  0001 L CNN
-	1    3850 2650
-	0    -1   -1   0
-$EndComp
-$Comp
-L Device:R_Small R?
-U 1 1 62E3EDFB
-P 3850 3000
-F 0 "R?" H 3909 3046 50  0000 L CNN
-F 1 "10k" H 3909 2955 50  0000 L CNN
-F 2 "" H 3850 3000 50  0001 C CNN
-F 3 "~" H 3850 3000 50  0001 C CNN
-	1    3850 3000
-	1    0    0    -1
-$EndComp
-$Comp
-L power:GND #PWR?
-U 1 1 62E3F633
-P 3850 3200
-F 0 "#PWR?" H 3850 2950 50  0001 C CNN
-F 1 "GND" H 3855 3027 50  0000 C CNN
-F 2 "" H 3850 3200 50  0001 C CNN
-F 3 "" H 3850 3200 50  0001 C CNN
-	1    3850 3200
-	1    0    0    -1
-$EndComp
-Wire Wire Line
-	3850 3200 3850 3100
-Wire Wire Line
-	3850 2900 3850 2850
-Wire Wire Line
-	2900 2550 3650 2550
-Wire Wire Line
-	4050 2550 4300 2550
+	4300 2550 4850 2550
 Connection ~ 4850 2550
-$Comp
-L Device:D_Zener D?
-U 1 1 62E421A4
-P 4300 2750
-F 0 "D?" V 4254 2829 50  0000 L CNN
-F 1 "D_Zener" V 4345 2829 50  0000 L CNN
-F 2 "" H 4300 2750 50  0001 C CNN
-F 3 "~" H 4300 2750 50  0001 C CNN
-	1    4300 2750
-	0    1    1    0
-$EndComp
-Wire Wire Line
-	4300 2900 3850 2900
-Connection ~ 3850 2900
-Wire Wire Line
-	4300 2600 4300 2550
-Connection ~ 4300 2550
-Wire Wire Line
-	4300 2550 4850 2550
+Connection ~ 8500 3250
+Wire Wire Line
+	8500 3250 8500 3350
+Wire Wire Line
+	8500 3250 8500 3050
+Wire Wire Line
+	6350 3250 8500 3250
+$Comp
+L Regulator_Switching:TPS5430DDA U2
+U 1 1 62DE4279
+P 5850 2750
+F 0 "U2" H 5850 3217 50  0000 C CNN
+F 1 "TPS5430DDA" H 5850 3126 50  0000 C CNN
+F 2 "Package_SO:TI_SO-PowerPAD-8_ThermalVias" H 5900 2400 50  0001 L CIN
+F 3 "http://www.ti.com/lit/ds/symlink/tps5430.pdf" H 5850 2750 50  0001 C CNN
+F 4 "C9864" H 5850 2750 50  0001 C CNN "LCSC PART #"
+	1    5850 2750
+	1    0    0    -1
+$EndComp
+Wire Wire Line
+	6350 2950 6350 3250
 $EndSCHEMATC

Commit message: fixed up some mistakes
Parts:
- C3: LCSC (none) -> C96446
- C4: LCSC (none) -> C57112
- C6: LCSC (none) -> C16133
- D4: LCSC (none) -> C64982
- L1: LCSC (none) -> C32375
- R12: LCSC (none) -> C25197
- R13: LCSC (none) -> C23189
- U2: LCSC (none) -> C9864
Changed lines of the file:
@@
 F 3 "~" H 4850 2800 50  0001 C CNN
 F 4 "C96446" H 4850 2800 50  0001 C CNN "LCSC PART #"
+F 5 "C96446" H 4850 2800 50  0001 C CNN "LCSC"
 	1    4850 2800
 	1    0    0    -1
@@
 F 3 "~" H 6700 2550 50  0001 C CNN
 F 4 "C57112" H 6700 2550 50  0001 C CNN "LCSC PART #"
+F 5 "C57112" H 6700 2550 50  0001 C CNN "LCSC"
 	1    6700 2550
 	0    1    1    0
@@
 F 3 "~" H 8500 2950 50  0001 C CNN
 F 4 "C25197" H 8500 2950 50  0001 C CNN "LCSC PART #"
+F 5 "C25197" H 8500 2950 50  0001 C CNN "LCSC"
 	1    8500 2950
 	1    0    0    -1
@@
 F 3 "~" H 8500 3450 50  0001 C CNN
 F 4 "C23189" H 8500 3450 50  0001 C CNN "LCSC PART #"
+F 5 "C23189" H 8500 3450 50  0001 C CNN "LCSC"
 	1    8500 3450
 	1    0    0    -1
@@
 F 3 "http://www.jameco.com/Jameco/Products/ProdDS/1538777.pdf" H 7350 2750 50  0001 C CNN
 F 4 "C64982" H 7350 2750 50  0001 C CNN "LCSC PART #"
+F 5 "C64982" H 7350 2750 50  0001 C CNN "LCSC"
 	1    7350 2750
 	0    1    1    0
@@
 F 3 "~" H 7800 2550 50  0001 C CNN
 F 4 "C32375" H 7800 2550 50  0001 C CNN "LCSC PART #"
+F 5 "C32375" H 7800 2550 50  0001 C CNN "LCSC"
 	1    7800 2550
 	0    -1   -1   0
@@
 F 3 "~" H 8100 2750 50  0001 C CNN
 F 4 "C16133" H 8100 2750 50  0001 C CNN "LCSC PART #"
+F 5 "C16133" H 8100 2750 50  0001 C CNN "LCSC"
 	1    8100 2750
 	1    0    0    -1
@@
 F 3 "http://www.ti.com/lit/ds/symlink/tps5430.pdf" H 5850 2750 50  0001 C CNN
 F 4 "C9864" H 5850 2750 50  0001 C CNN "LCSC PART #"
+F 5 "C9864" H 5850 2750 50  0001 C CNN "LCSC"
 	1    5850 2750
 	1    0    0    -1
